Commit message: created spawn.launch changed color for gazebo

File: robotarm_description/urdf/materials.xacro (robot description, xacro)
@@ -4,3 +4,27 @@
   <color rgba="0.700 0.700 0.700 1.000"/>
 </material>
+<material name="black">
+  <color rgba="0.0 0.0 0.0 1.0"/>
+</material>
+<material name="blue">
+  <color rgba="0.0 0.0 0.8 1.0"/>
+</material>
+<material name="green">
+  <color rgba="0.0 1.0 0.0 1.0"/>
+</material>
+<material name="grey">
+  <color rgba="0.4 0.4 0.4 1.0"/>
+</material>
+<material name="orange">
+  <color rgba="${255/255} ${108/255} ${10/255} 1.0"/>
+</material>
+<material name="brown">
+  <color rgba="${222/255} ${207/255} ${195/255} 1.0"/>
+</material>
+<material name="red">
+  <color rgba="0.4 0.2 0.2 1.0"/>
+</material>
+<material name="white">
+  <color rgba="0.8 0.8 0.8 1.0"/>
+</material>
 </robot>

File: robotarm_description/urdf/robotarm.xacro (robot description, xacro)
@@ -15,5 +15,5 @@
       <mesh filename="package://robotarm_description/meshes/base_link.stl" scale="0.001 0.001 0.001"/>
     </geometry>
-    <material name="silver"/>
+    <material name="black"/>
   </visual>
   <collision>
@@ -35,5 +35,5 @@
       <mesh filename="package://robotarm_description/meshes/link_1_1.stl" scale="0.001 0.001 0.001"/>
     </geometry>
-    <material name="silver"/>
+    <material name="grey"/>
   </visual>
   <collision>
@@ -55,5 +55,5 @@
       <mesh filename="package://robotarm_description/meshes/link_2_1.stl" scale="0.001 0.001 0.001"/>
     </geometry>
-    <material name="silver"/>
+    <material name="black"/>
   </visual>
   <collision>
@@ -75,5 +75,5 @@
       <mesh filename="package://robotarm_description/meshes/link_3_1.stl" scale="0.001 0.001 0.001"/>
     </geometry>
-    <material name="silver"/>
+    <material name="grey"/>
   </visual>
   <collision>
@@ -95,5 +95,5 @@
       <mesh filename="package://robotarm_description/meshes/link_4_1.stl" scale="0.001 0.001 0.001"/>
     </geometry>
-    <material name="silver"/>
+    <material name="white"/>
   </visual>
   <collision>
@@ -115,5 +115,5 @@
       <mesh filename="package://robotarm_description/meshes/link_5_1.stl" scale="0.001 0.001 0.001"/>
     </geometry>
-    <material name="silver"/>
+    <material name="grey"/>
   </visual>
   <collision>
@@ -135,5 +135,5 @@
       <mesh filename="package://robotarm_description/meshes/link_6_1.stl" scale="0.001 0.001 0.001"/>
     </geometry>
-    <material name="silver"/>
+    <material name="white"/>
   </visual>
   <collision>
@@ -155,5 +155,5 @@
       <mesh filename="package://robotarm_description/meshes/link_7_1.stl" scale="0.001 0.001 0.001"/>
     </geometry>
-    <material name="silver"/>
+    <material name="grey"/>
   </visual>
   <collision>
@@ -175,5 +175,5 @@
       <mesh filename="package://robotarm_description/meshes/link_8_1.stl" scale="0.001 0.001 0.001"/>
     </geometry>
-    <material name="silver"/>
+    <material name="black"/>
   </visual>
   <collision>
@@ -195,5 +195,5 @@
       <mesh filename="package://robotarm_description/meshes/link_9_1.stl" scale="0.001 0.001 0.001"/>
     </geometry>
-    <material name="silver"/>
+    <material name="white"/>
   </visual>
   <collision>
@@ -215,5 +215,5 @@
       <mesh filename="package://robotarm_description/meshes/link_10_1.stl" scale="0.001 0.001 0.001"/>
     </geometry>
-    <material name="silver"/>
+    <material name="black"/>
   </visual>
   <collision>
@@ -235,5 +235,5 @@
       <mesh filename="package://robotarm_description/meshes/link_11_1.stl" scale="0.001 0.001 0.001"/>
     </geometry>
-    <material name="silver"/>
+    <material name="white"/>
   </visual>
   <collision>
@@ -255,5 +255,5 @@
       <mesh filename="package://robotarm_description/meshes/link_12_1.stl" scale="0.001 0.001 0.001"/>
     </geometry>
-    <material name="silver"/>
+    <material name="black"/>
   </visual>
   <collision>
@@ -275,5 +275,5 @@
       <mesh filename="package://robotarm_description/meshes/link_13_1.stl" scale="0.001 0.001 0.001"/>
     </geometry>
-    <material name="silver"/>
+    <material name="black"/>
   </visual>
   <collision>
