Commit message: world modified parameters adjusted

File: robotarm/robotarm_description/urdf/robotarm.xacro (robot description, xacro)
@@ -103,5 +103,5 @@
     </gazebo>
     <gazebo reference="link_1_1">
-        <material>Gazebo/Grey</material>
+        <material>Gazebo/FlatBlack</material>
         <mu1>0.2</mu1>
         <mu2>0.2</mu2>
@@ -115,5 +115,5 @@
     </gazebo>
     <gazebo reference="link_3_1">
-        <material>Gazebo/Grey</material>
+        <material>Gazebo/FlatBlack</material>
         <mu1>0.2</mu1>
         <mu2>0.2</mu2>
@@ -121,5 +121,5 @@
     </gazebo>
     <gazebo reference="link_4_1">
-        <material>$Gazebo/White</material>
+        <material>Gazebo/White</material>
         <mu1>0.2</mu1>
         <mu2>0.2</mu2>
@@ -127,5 +127,5 @@
     </gazebo>
     <gazebo reference="link_5_1">
-        <material>Gazebo/Grey</material>
+        <material>Gazebo/FlatBlack</material>
         <mu1>0.2</mu1>
         <mu2>0.2</mu2>
@@ -139,5 +139,5 @@
     </gazebo>
     <gazebo reference="link_7_1">
-        <material>Gazebo/Grey</material>
+        <material>Gazebo/FlatBlack</material>
         <mu1>0.2</mu1>
         <mu2>0.2</mu2>
@@ -169,5 +169,5 @@
     </gazebo>
     <gazebo reference="link_12_1">
-        <material>Gazebo/Grey</material>
+        <material>Gazebo/FlatBlack</material>
         <mu1>0.2</mu1>
         <mu2>0.2</mu2>
@@ -181,5 +181,5 @@
     </gazebo>
     <gazebo reference="grabber_1">
-        <material>Gazebo/Grey</material>
+        <material>Gazebo/FlatBlack</material>
         <mu1>0.2</mu1>
         <mu2>0.2</mu2>
